File: ASD2411.brd (EAGLE design)
At the start: 22.5 x 22.5 mm, 24 parts, among them J1 DF12-32-DP, J2 DF12-32-DS

Commit message: Updated to Rev 4
Other:
- board text added: "4"
- board text added: "ASD2411 - Rev4"
- board text added: "LED 16 TinyShield"
- board text removed: "3"
- board text removed: "ASD2411"
- board text removed: "REV 3"
- board text removed: "TinyShield - LED"
