File: design_files/ASD2411.brd (EAGLE design)
At the start: 22.5 x 22.5 mm, 24 parts, among them J1 DF12-32-DP, J2 DF12-32-DS

Commit message: update format and rev
Other:
- board size 22.5 x 22.5 mm -> 22.5 x 21.3 mm
- board text added: "5"
- board text added: "ASD2411 - Rev5"
- board text added: "TinyCircuits.com"
- board text added: "^ V-SCORE EDGE ALONG OUTLINE ^"
- board text removed: "4"
- board text removed: "ASD2411 - Rev4"
- board text removed: "Tiny-Circuits.com"
